Commit message: Adjust rover sensor and RViz defaults

File: ros2_ws/src/rover_description/urdf/student_rover.urdf.xacro (robot description, xacro)
@@ -64,5 +64,5 @@
     <parent link="base_link"/>
     <child link="lidar_link"/>
-    <origin xyz="0 0 ${body_z/2.0 + lidar_box_z/2.0}" rpy="0 0 0"/>
+    <origin xyz="${body_x/2.0 + lidar_box_x/2.0} 0 ${-body_z/2.0 - lidar_box_z/0.7}" rpy="0 0.0 0"/> #TODO: Adjust the lidar pitch and position to be more useful for obstacle detection.
   </joint>
   <link name="front_camera_link">
